File: V-00724-00.brd (EAGLE design)
At the start: 56 x 37.5 mm, 19 parts, among them IC1 MEGA8-AI, IC2 MAX481CSA, Q1 14.7456MHz

Commit message: v1.1.0.1
Parts:
- removed K1, K2: (no value), #PaJa_konektory:PSH02-04W
- added K3: (no value), #PaJa_konektory:PSH02-02P
- added Q2: N-HEXFET_SOT323-IRLL014N, transistor-power:SOT223
- added R4: 10k, #PaJa_31:1206
- added REL1: RELSIA?, #PaJa_31:RELSIA
- CAN1: value CAN_9V_/0 -> CAN_9V_/90; device #PaJa_konektory:CAN9V -> #PaJa_konektory:CAN9V/90
- moved U$1 125.6 mm to (38.8, 12.9), turned to 90 degrees
- moved C6 117.5 mm to (44.0, 14.6), turned to 90 degrees
- moved C5 117.1 mm to (48.6, 14.6), turned to 90 degrees
- moved D1 112.2 mm to (47.6, 25.3), flipped to the bottom, turned to 90 degrees
- moved IO2 106.8 mm to (46.3, 12.8), flipped to the bottom, turned to 180 degrees
- moved CAN1 87.5 mm to (29.4, 27.1)
- moved C4 85.0 mm to (34.4, 23.3), flipped to the bottom, turned to 270 degrees
- moved C3 79.6 mm to (29.4, 23.3), flipped to the bottom, turned to 270 degrees
- moved Q1 71.3 mm to (31.9, 20.2), turned to 180 degrees
- moved C2 65.0 mm to (39.5, 1.70), flipped to the bottom
- moved C1 56.2 mm to (36.3, 3.90), flipped to the bottom
- moved R3 53.3 mm to (20.7, 11.3), flipped to the bottom, turned to 270 degrees
- moved IO1 49.2 mm to (30.8, 4.10), flipped to the bottom, turned to 180 degrees
- moved R1 45.6 mm to (23.3, 3.30), flipped to the bottom, turned to 270 degrees
- moved R2 45.5 mm to (20.7, 3.30), flipped to the bottom, turned to 90 degrees
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Connections:
- removed net N$10: CAN1.6
- removed net N$12: CAN1.8
- removed net N$14: IC1.23, K1.1
- removed net N$15: IC1.24, K1.2
- removed net N$16: IC1.25, K1.3
- removed net N$17: IC1.26, K1.4
- removed net N$18: IC1.2, K2.1
- removed net N$19: IC1.9, K2.2
- removed net N$20: IC1.10, K2.3
- removed net N$23: IC1.11, K2.4
- removed net N$3: CAN1.1
- removed net N$4: CAN1.2
- removed net N$8: CAN1.4
- removed net N$9: CAN1.5
- new net N$21: IC1.27, Q2.1, R4.2
- new net N$24: Q2.4, REL1.-5
- new net N$27: K3.1, REL1.7
- net +24V: now also REL1.1
- net +24V_OUT: now also CAN1.1
- net +5V: now also CAN1.4, REL1.+3
- net BUS_A: now also CAN1.6
- net BUS_B: now also CAN1.8
- net GND: now also CAN1.2, CAN1.5, K3.2, Q2.3, R4.1
Routing:
- net +5V: track 0.00 -> 79.3 mm, vias 0 -> 2
- net N$24: track 0.00 -> 48.8 mm, vias 0 -> 1
- net +24V: track 0.00 -> 32.0 mm
- net N$6: track 0.00 -> 28.7 mm
- net BUS_A: track 0.00 -> 22.6 mm, vias 0 -> 1
- net RESET: track 0.00 -> 22.5 mm, vias 0 -> 1
- net N$21: track 0.00 -> 18.2 mm
- net BUS_B: track 0.00 -> 17.9 mm
- net +24V_OUT: track 0.00 -> 16.0 mm
- net N$1: track 0.00 -> 15.1 mm
- net P_MOSI: track 0.00 -> 12.7 mm
- net RS485_EN: track 0.00 -> 10.9 mm
- net N$27: track 0.00 -> 10.8 mm
- net RS485_TX: track 0.00 -> 9.18 mm, vias 0 -> 2
- net P_SCK: track 0.00 -> 6.87 mm
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- added copper zone on layer 16, net +5V
- added copper zone on layer 1, net GND
- added copper zone on layer 16, net GND
Other:
- board size 56 x 37.5 mm -> 62 x 43.5 mm
- board text added: "V-00724-00 Author: LN 11.12.2015"
- board text removed: "USB <-> RS485"

Commit message: v1.1.0.2
Parts:
- moved Q1 0.20 mm to (31.9, 20.0), flipped to the bottom, turned to 0 degrees
Changed lines of the file:
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@@
 <layer number="14" name="Route14" color="1" fill="6" visible="no" active="yes"/>
 <layer number="15" name="Route15" color="4" fill="6" visible="no" active="yes"/>
-<layer number="16" name="Bottom" color="4" fill="1" visible="no" active="yes"/>
+<layer number="16" name="Bottom" color="4" fill="1" visible="yes" active="yes"/>
 <layer number="17" name="Pads" color="2" fill="1" visible="yes" active="yes"/>
 <layer number="18" name="Vias" color="2" fill="1" visible="yes" active="yes"/>
-<layer number="19" name="Unrouted" color="6" fill="1" visible="no" active="yes"/>
+<layer number="19" name="Unrouted" color="6" fill="1" visible="yes" active="yes"/>
 <layer number="20" name="Dimension" color="15" fill="1" visible="yes" active="yes"/>
-<layer number="21" name="tPlace" color="7" fill="1" visible="no" active="yes"/>
-<layer number="22" name="bPlace" color="7" fill="1" visible="no" active="yes"/>
-<layer number="23" name="tOrigins" color="15" fill="1" visible="no" active="yes"/>
-<layer number="24" name="bOrigins" color="15" fill="1" visible="no" active="yes"/>
-<layer number="25" name="tNames" color="7" fill="1" visible="no" active="yes"/>
-<layer number="26" name="bNames" color="7" fill="1" visible="no" active="yes"/>
-<layer number="27" name="tValues" color="7" fill="1" visible="no" active="yes"/>
-<layer number="28" name="bValues" color="7" fill="1" visible="no" active="yes"/>
+<layer number="21" name="tPlace" color="7" fill="1" visible="yes" active="yes"/>
+<layer number="22" name="bPlace" color="7" fill="1" visible="yes" active="yes"/>
+<layer number="23" name="tOrigins" color="15" fill="1" visible="yes" active="yes"/>
+<layer number="24" name="bOrigins" color="15" fill="1" visible="yes" active="yes"/>
+<layer number="25" name="tNames" color="7" fill="1" visible="yes" active="yes"/>
+<layer number="26" name="bNames" color="7" fill="1" visible="yes" active="yes"/>
+<layer number="27" name="tValues" color="7" fill="1" visible="yes" active="yes"/>
+<layer number="28" name="bValues" color="7" fill="1" visible="yes" active="yes"/>
 <layer number="29" name="tStop" color="7" fill="3" visible="no" active="yes"/>
 <layer number="30" name="bStop" color="7" fill="6" visible="no" active="yes"/>
@@
 <element name="R3" library="#PaJa_31" package="1206" value="10k" x="20.7" y="11.3" rot="MR270"/>
 <element name="C2" library="#PaJa_31" package="1206" value="10uF" x="39.5" y="1.7" rot="MR0"/>
-<element name="Q1" library="#PaJa_31" package="HC-49U" value="14.7456MHz" x="31.9" y="20.2" rot="R180"/>
+<element name="Q1" library="#PaJa_31" package="HC-49U" value="14.7456MHz" x="31.9" y="20" rot="MR0"/>
 <element name="C3" library="#PaJa_31" package="0805" value="27nF" x="29.4" y="23.3" rot="MR270"/>
 <element name="C4" library="#PaJa_31" package="0805" value="27nF" x="34.4" y="23.3" rot="MR270"/>
@@
 <contactref element="C3" pad="2"/>
 <contactref element="Q1" pad="2"/>
-<wire x1="31.5" y1="16.7926" x2="31.5" y2="18.06" width="0.4064" layer="16"/>
-<wire x1="31.5" y1="18.06" x2="29.36" y2="20.2" width="0.4064" layer="16"/>
-<wire x1="29.36" y1="20.2" x2="29.36" y2="22.3075" width="0.4064" layer="16"/>
+<wire x1="31.5" y1="16.7926" x2="31.5" y2="17.86" width="0.4064" layer="16"/>
+<wire x1="31.5" y1="17.86" x2="29.36" y2="20" width="0.4064" layer="16"/>
+<wire x1="29.36" y1="20" x2="29.36" y2="22.3075" width="0.4064" layer="16"/>
 <wire x1="29.36" y1="22.3075" x2="29.4" y2="22.3475" width="0.4064" layer="16"/>
 </signal>
@@
 <contactref element="Q1" pad="1"/>
 <contactref element="C4" pad="2"/>
-<wire x1="32.3" y1="16.7926" x2="32.3" y2="18.06" width="0.4064" layer="16"/>
-<wire x1="32.3" y1="18.06" x2="34.44" y2="20.2" width="0.4064" layer="16"/>
-<wire x1="34.44" y1="20.2" x2="34.44" y2="22.3075" width="0.4064" layer="16"/>
+<wire x1="32.3" y1="16.7926" x2="32.3" y2="17.86" width="0.4064" layer="16"/>
+<wire x1="32.3" y1="17.86" x2="34.44" y2="20" width="0.4064" layer="16"/>
+<wire x1="34.44" y1="20" x2="34.44" y2="22.3075" width="0.4064" layer="16"/>
 <wire x1="34.44" y1="22.3075" x2="34.4" y2="22.3475" width="0.4064" layer="16"/>
 </signal>
