File: V-00724-00.sch (EAGLE design)
At the start: 19 parts, among them IC1 MEGA8-AI, IC2 MAX481CSA, Q1 14.7456MHz

Commit message: v1.1.0.1
Parts:
- removed K1, K2: (no value), #PaJa_konektory:PSH02-04W
- added K3: (no value), #PaJa_konektory:PSH02-02P
- added Q2: N-HEXFET_SOT323-IRLL014N, transistor-power:N-HEXFET_SOT323-IRLL014N
- added R4: 10k, #PaJa_31:R_1206
- added REL1: RELSIA, #PaJa_31:RELSIA
- CAN1: value CAN_9V_/0 -> CAN_9V_/90; device #PaJa_konektory:CAN_9V_/0 -> #PaJa_konektory:CAN_9V_/90
Connections:
- removed net N$10: CAN1.6
- removed net N$12: CAN1.8
- removed net N$14: IC1.PC0(ADC0), K1.1
- removed net N$15: IC1.PC1(ADC1), K1.2
- removed net N$16: IC1.PC2(ADC2), K1.3
- removed net N$17: IC1.PC3(ADC3), K1.4
- removed net N$18: IC1.PD4(XCK/T0), K2.1
- removed net N$19: IC1.PD5(T1), K2.2
- removed net N$20: IC1.PD6(AIN0), K2.3
- removed net N$23: IC1.PD7(AIN1), K2.4
- removed net N$3: CAN1.1
- removed net N$4: CAN1.2
- removed net N$8: CAN1.4
- removed net N$9: CAN1.5
- new net N$21: IC1.PC4(ADC4/SDA), Q2.G, R4.2
- new net N$24: Q2.D, REL1CIVKA.C-
- new net N$27: K3.1, REL1SPIN.2
- net +24V: now also REL1SPIN.1
- net +24V_OUT: now also CAN1.1
- net +5V: now also CAN1.4, REL1CIVKA.C+
- net BUS_A: now also CAN1.6
- net BUS_B: now also CAN1.8
- net GND: now also CAN1.2, CAN1.5, K3.2, Q2.S, R4.1
Other:
- moved on the sheet: CAN1

Commit message: v.2.0
Other:
- note added: "Spatny ISP!!!!!"
- moved on the sheet: CAN1
Changed lines of the file:
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@@
 RS485 -&gt; 5TTL</text>
 <text x="246.38" y="5.08" size="2.54" layer="94">00</text>
+<text x="170.18" y="86.36" size="1.778" layer="97">Spatny ISP!!!!! </text>
 </plain>
 <instances>
@@
 <instance part="C3" gate="C" x="25.4" y="73.66" rot="R90"/>
 <instance part="C4" gate="C" x="43.18" y="73.66" rot="R90"/>
-<instance part="CAN1" gate="CAN" x="218.44" y="66.04"/>
+<instance part="CAN1" gate="CAN" x="223.52" y="73.66" rot="R270"/>
 <instance part="D1" gate="G$1" x="124.46" y="167.64"/>
 <instance part="IO2" gate="IO" x="152.4" y="167.64"/>
@@
 <segment>
 <pinref part="CAN1" gate="CAN" pin="6"/>
-<wire x1="210.82" y1="63.5" x2="210.82" y2="55.88" width="0.1524" layer="91"/>
-<label x="210.82" y="55.88" size="1.016" layer="95" font="vector" ratio="10" rot="R270" xref="yes"/>
+<wire x1="220.98" y1="81.28" x2="213.36" y2="81.28" width="0.1524" layer="91"/>
+<label x="213.36" y="81.28" size="1.016" layer="95" font="vector" ratio="10" rot="R180" xref="yes"/>
 </segment>
 </net>
@@
 <segment>
 <pinref part="CAN1" gate="CAN" pin="8"/>
-<wire x1="220.98" y1="63.5" x2="220.98" y2="55.88" width="0.1524" layer="91"/>
-<label x="220.98" y="55.88" size="1.016" layer="95" font="vector" ratio="10" rot="R270" xref="yes"/>
+<wire x1="220.98" y1="71.12" x2="213.36" y2="71.12" width="0.1524" layer="91"/>
+<label x="213.36" y="71.12" size="1.016" layer="95" font="vector" ratio="10" rot="R180" xref="yes"/>
 </segment>
 </net>
@@
 <segment>
 <pinref part="CAN1" gate="CAN" pin="4"/>
-<wire x1="223.52" y1="68.58" x2="223.52" y2="76.2" width="0.1524" layer="91"/>
-<label x="223.52" y="76.2" size="1.016" layer="95" font="vector" ratio="10" rot="R90" xref="yes"/>
+<wire x1="226.06" y1="68.58" x2="233.68" y2="68.58" width="0.1524" layer="91"/>
+<label x="233.68" y="68.58" size="1.016" layer="95" font="vector" ratio="10" xref="yes"/>
 </segment>
 </net>
@@
 <segment>
 <pinref part="CAN1" gate="CAN" pin="5"/>
-<wire x1="228.6" y1="68.58" x2="228.6" y2="76.2" width="0.1524" layer="91"/>
-<label x="228.6" y="76.2" size="1.016" layer="95" font="vector" ratio="10" rot="R90" xref="yes"/>
+<wire x1="226.06" y1="63.5" x2="233.68" y2="63.5" width="0.1524" layer="91"/>
+<label x="233.68" y="63.5" size="1.016" layer="95" font="vector" ratio="10" xref="yes"/>
 </segment>
 <segment>
 <pinref part="CAN1" gate="CAN" pin="2"/>
-<wire x1="213.36" y1="68.58" x2="213.36" y2="76.2" width="0.1524" layer="91"/>
-<label x="213.36" y="76.2" size="1.016" layer="95" font="vector" ratio="10" rot="R90" xref="yes"/>
+<wire x1="226.06" y1="78.74" x2="233.68" y2="78.74" width="0.1524" layer="91"/>
+<label x="233.68" y="78.74" size="1.016" layer="95" font="vector" ratio="10" xref="yes"/>
 </segment>
 </net>
@@
 <segment>
 <pinref part="CAN1" gate="CAN" pin="3"/>
-<wire x1="218.44" y1="68.58" x2="218.44" y2="76.2" width="0.1524" layer="91"/>
-<label x="218.44" y="76.2" size="1.016" layer="95" font="vector" ratio="10" rot="R90" xref="yes"/>
+<wire x1="226.06" y1="73.66" x2="233.68" y2="73.66" width="0.1524" layer="91"/>
+<label x="233.68" y="73.66" size="1.016" layer="95" font="vector" ratio="10" xref="yes"/>
 </segment>
 </net>
@@
 <segment>
 <pinref part="CAN1" gate="CAN" pin="7"/>
-<wire x1="215.9" y1="63.5" x2="215.9" y2="55.88" width="0.1524" layer="91"/>
-<label x="215.9" y="55.88" size="1.016" layer="95" font="vector" ratio="10" rot="R270" xref="yes"/>
+<wire x1="220.98" y1="76.2" x2="213.36" y2="76.2" width="0.1524" layer="91"/>
+<label x="213.36" y="76.2" size="1.016" layer="95" font="vector" ratio="10" rot="R180" xref="yes"/>
 </segment>
 </net>
@@
 <segment>
 <pinref part="CAN1" gate="CAN" pin="9"/>
-<wire x1="226.06" y1="63.5" x2="226.06" y2="55.88" width="0.1524" layer="91"/>
-<label x="226.06" y="55.88" size="1.016" layer="95" font="vector" ratio="10" rot="R270" xref="yes"/>
+<wire x1="220.98" y1="66.04" x2="213.36" y2="66.04" width="0.1524" layer="91"/>
+<label x="213.36" y="66.04" size="1.016" layer="95" font="vector" ratio="10" rot="R180" xref="yes"/>
 </segment>
 </net>
@@
 <segment>
 <pinref part="CAN1" gate="CAN" pin="1"/>
-<wire x1="208.28" y1="68.58" x2="208.28" y2="76.2" width="0.1524" layer="91"/>
-<label x="208.28" y="76.2" size="1.016" layer="95" font="vector" ratio="10" rot="R90" xref="yes"/>
-</segment>
-</net>
+<wire x1="226.06" y1="83.82" x2="233.68" y2="83.82" width="0.1524" layer="91"/>
+<label x="233.68" y="83.82" size="1.016" layer="95" font="vector" ratio="10" xref="yes"/>
+</segment>
+</net>
